File: ApogeoShield.kicad_pcb (KiCad board)
At the start: 2 copper layers, 68.6 x 53.3 mm, 28 parts, among them J1 Conn_02x03_Odd_Even, J2 Conn_Coaxial, J4 Conn_01x06_Pin, J5 Conn_01x06_Pin, J6 Conn_01x08_Pin, J7 Conn_01x08_Pin, P1 USB_C_Plug_USB2.0

Commit message: Release 1.1b
Parts:
- added REF**: OSHW-Logo2_7.3x6mm_SilkScreen, Symbol:OSHW-Logo2_7.3x6mm_SilkScreen, F.Cu at (137.2, 96.5)
