File: ApogeoShield.kicad_sch (KiCad schematic)
At the start: 28 parts, among them J1 Conn_02x03_Odd_Even, J2 Conn_Coaxial, J4 Conn_01x06_Pin, J5 Conn_01x06_Pin, J6 Conn_01x08_Pin, J7 Conn_01x08_Pin, P1 USB_C_Plug_USB2.0

Commit message: Release 1.1b
Other:
- note added: "1.0 - 31/10/2023 First version. 1.1 - 14/11/2023 Added configuration of SS, RST and D0 pins via resistor placement. 1.1b - 30/05/2023 Re-added Company logo (internal); added OSHW logo"
- note removed: "1.0 - 31/10/2023 First version. 1.1 - 14/11/2023 Added configuration of SS, RST and D0 pins via resistor placement."
- title: Nodo Arduino -> ApogeoShield
Changed lines of the file:
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@@
 	(paper "A4")
 	(title_block
-		(title "Nodo Arduino")
+		(title "ApogeoShield")
 		(date "2023-11-14")
 		(rev "1.1")
@@
 		)
 	)
-	(text "1.0 - 31/10/2023 First version.\n1.1 - 14/11/2023 Added configuration of SS, RST and D0 pins via resistor placement.\n"
+	(text "1.0 - 31/10/2023 First version.\n1.1 - 14/11/2023 Added configuration of SS, RST and D0 pins via resistor placement.\n1.1b - 30/05/2023 Re-added Company logo (internal); added OSHW logo"
 		(exclude_from_sim no)
 		(at 21.59 113.03 0)
@@
 		)
 		(instances
-			(project "Nodo_A_HW"
+			(project "ApogeoShield"
 				(path "/1d67b07b-d997-41b7-9a0a-a4770aa9f862"
 					(reference "#PWR03")
@@
 		)
 		(instances
-			(project "Nodo_A_HW"
+			(project "ApogeoShield"
 				(path "/1d67b07b-d997-41b7-9a0a-a4770aa9f862"
 					(reference "RS4")
@@
 		)
 		(instances
-			(project "Nodo_A_HW"
+			(project "ApogeoShield"
 				(path "/1d67b07b-d997-41b7-9a0a-a4770aa9f862"
 					(reference "RR2")
@@
 		)
 		(instances
-			(project "Nodo_A_HW"
+			(project "ApogeoShield"
 				(path "/1d67b07b-d997-41b7-9a0a-a4770aa9f862"
 					(reference "RI2")
@@
 		)
 		(instances
-			(project "Nodo_A_HW"
+			(project "ApogeoShield"
 				(path "/1d67b07b-d997-41b7-9a0a-a4770aa9f862"
 					(reference "#PWR06")
@@
 		)
 		(instances
-			(project "Nodo_A_HW"
+			(project "ApogeoShield"
 				(path "/1d67b07b-d997-41b7-9a0a-a4770aa9f862"
 					(reference "R6")
@@
 		)
 		(instances
-			(project "Nodo_A_HW"
+			(project "ApogeoShield"
 				(path "/1d67b07b-d997-41b7-9a0a-a4770aa9f862"
 					(reference "RO2")
@@
 		)
 		(instances
-			(project "Nodo_A_HW"
+			(project "ApogeoShield"
 				(path "/1d67b07b-d997-41b7-9a0a-a4770aa9f862"
 					(reference "#PWR08")
@@
 		)
 		(instances
-			(project "Nodo_A_HW"
+			(project "ApogeoShield"
 				(path "/1d67b07b-d997-41b7-9a0a-a4770aa9f862"
 					(reference "J7")
@@
 		)
 		(instances
-			(project "Nodo_A_HW"
+			(project "ApogeoShield"
 				(path "/1d67b07b-d997-41b7-9a0a-a4770aa9f862"
 					(reference "MOD1")
@@
 		)
 		(instances
-			(project "Nodo_A_HW"
+			(project "ApogeoShield"
 				(path "/1d67b07b-d997-41b7-9a0a-a4770aa9f862"
 					(reference "RC1")
@@
 		)
 		(instances
-			(project "Nodo_A_HW"
+			(project "ApogeoShield"
 				(path "/1d67b07b-d997-41b7-9a0a-a4770aa9f862"
 					(reference "R7")
@@
 		)
 		(instances
-			(project "Nodo_A_HW"
+			(project "ApogeoShield"
 				(path "/1d67b07b-d997-41b7-9a0a-a4770aa9f862"
 					(reference "#PWR05")
@@
 		)
 		(instances
-			(project "Nodo_A_HW"
+			(project "ApogeoShield"
 				(path "/1d67b07b-d997-41b7-9a0a-a4770aa9f862"
 					(reference "RS2")
@@
 		)
 		(instances
-			(project "Nodo_A_HW"
+			(project "ApogeoShield"
 				(path "/1d67b07b-d997-41b7-9a0a-a4770aa9f862"
 					(reference "#PWR010")
@@
 		)
 		(instances
-			(project "Nodo_A_HW"
+			(project "ApogeoShield"
 				(path "/1d67b07b-d997-41b7-9a0a-a4770aa9f862"
 					(reference "RO1")
@@
 		)
 		(instances
-			(project "Nodo_A_HW"
+			(project "ApogeoShield"
 				(path "/1d67b07b-d997-41b7-9a0a-a4770aa9f862"
 					(reference "#PWR07")
@@
 		)
 		(instances
-			(project "Nodo_A_HW"
+			(project "ApogeoShield"
 				(path "/1d67b07b-d997-41b7-9a0a-a4770aa9f862"
 					(reference "RS1")
@@
 		)
 		(instances
-			(project "Nodo_A_HW"
+			(project "ApogeoShield"
 				(path "/1d67b07b-d997-41b7-9a0a-a4770aa9f862"
 					(reference "RR3")
@@
 		)
 		(instances
-			(project "Nodo_A_HW"
+			(project "ApogeoShield"
 				(path "/1d67b07b-d997-41b7-9a0a-a4770aa9f862"
 					(reference "#PWR01")
@@
 		)
 		(instances
-			(project "Nodo_A_HW"
+			(project "ApogeoShield"
 				(path "/1d67b07b-d997-41b7-9a0a-a4770aa9f862"
 					(reference "RS5")
@@
 		)
 		(instances
-			(project "Nodo_A_HW"
+			(project "ApogeoShield"
 				(path "/1d67b07b-d997-41b7-9a0a-a4770aa9f862"
 					(reference "RC2")
@@
 		)
 		(instances
-			(project "Nodo_A_HW"
+			(project "ApogeoShield"
 				(path "/1d67b07b-d997-41b7-9a0a-a4770aa9f862"
 					(reference "RI1")
@@
 		)
 		(instances
-			(project "Nodo_A_HW"
+			(project "ApogeoShield"
 				(path "/1d67b07b-d997-41b7-9a0a-a4770aa9f862"
 					(reference "J1")
@@
 		)
 		(instances
-			(project "Nodo_A_HW"
+			(project "ApogeoShield"
 				(path "/1d67b07b-d997-41b7-9a0a-a4770aa9f862"
 					(reference "R9")
@@
 		)
 		(instances
-			(project "Nodo_A_HW"
+			(project "ApogeoShield"
 				(path "/1d67b07b-d997-41b7-9a0a-a4770aa9f862"
 					(reference "J5")
@@
 		)
 		(instances
-			(project "Nodo_A_HW"
+			(project "ApogeoShield"
 				(path "/1d67b07b-d997-41b7-9a0a-a4770aa9f862"
 					(reference "J2")
@@
 		)
 		(instances
-			(project "Nodo_A_HW"
+			(project "ApogeoShield"
 				(path "/1d67b07b-d997-41b7-9a0a-a4770aa9f862"
 					(reference "P1")
@@
 		)
 		(instances
-			(project "Nodo_A_HW"
+			(project "ApogeoShield"
 				(path "/1d67b07b-d997-41b7-9a0a-a4770aa9f862"
 					(reference "RR1")
@@
 		)
 		(instances
-			(project "Nodo_A_HW"
+			(project "ApogeoShield"
 				(path "/1d67b07b-d997-41b7-9a0a-a4770aa9f862"
 					(reference "#PWR04")
@@
 		)
 		(instances
-			(project "Nodo_A_HW"
+			(project "ApogeoShield"
 				(path "/1d67b07b-d997-41b7-9a0a-a4770aa9f862"
 					(reference "#PWR02")
@@
 		)
 		(instances
-			(project "Nodo_A_HW"
+			(project "ApogeoShield"
 				(path "/1d67b07b-d997-41b7-9a0a-a4770aa9f862"
 					(reference "RD1")
@@
 		)
 		(instances
-			(project "Nodo_A_HW"
+			(project "ApogeoShield"
 				(path "/1d67b07b-d997-41b7-9a0a-a4770aa9f862"
 					(reference "RS3")
@@
 		)
 		(instances
-			(project "Nodo_A_HW"
+			(project "ApogeoShield"
 				(path "/1d67b07b-d997-41b7-9a0a-a4770aa9f862"
 					(reference "#PWR09")
@@
 		)
 		(instances
-			(project "Nodo_A_HW"
+			(project "ApogeoShield"
 				(path "/1d67b07b-d997-41b7-9a0a-a4770aa9f862"
 					(reference "J4")
@@
 		)
 		(instances
-			(project "Nodo_A_HW"
+			(project "ApogeoShield"
 				(path "/1d67b07b-d997-41b7-9a0a-a4770aa9f862"
 					(reference "R8")
@@
 		)
 		(instances
-			(project "Nodo_A_HW"
+			(project "ApogeoShield"
 				(path "/1d67b07b-d997-41b7-9a0a-a4770aa9f862"
 					(reference "RD2")
@@
 		)
 		(instances
-			(project "Nodo_A_HW"
+			(project "ApogeoShield"
 				(path "/1d67b07b-d997-41b7-9a0a-a4770aa9f862"
 					(reference "J6")
